Commit message: change the drive strategy

File: bluecrescent_description/urdf/bluecrescent.urdf (robot description, URDF)
Before this commit: robot bluecrescent, 20 links, 19 joints
Joints:
- joint head_roll: limit lower=-0.5 upper=0.5 effort=1000.0 velocity=0.5 -> lower=-0.4 upper=0.4 effort=1000.0 velocity=0.2
- joint head_yaw: limit lower=-0.5 upper=0.5 effort=1000.0 velocity=0.5 -> lower=-0.4 upper=0.4 effort=1000.0 velocity=0.2
